Commit message: Add velocity limits to wheel joints in URDF

File: contributions/urdf-gazebo-sim/alvarosamudio/oomwoo_gazebo/urdf/robot.urdf.xacro (robot description, xacro)
@@ -72,5 +72,5 @@
     <origin xyz="0 ${wheel_base/2} ${wheel_diameter/2 - floor_clearance}" rpy="-${pi/2} 0 0"/>
     <axis xyz="0 0 1"/>
-    <limit effort="${motor_stall_torque}"/>
+    <limit effort="${motor_stall_torque}" velocity="1.0"/>
   </joint>
   <link name="wheel_left_link">
@@ -93,5 +93,5 @@
     <origin xyz="0 ${-wheel_base/2} ${wheel_diameter/2 - floor_clearance}" rpy="-${pi/2} 0 0"/>
     <axis xyz="0 0 1"/>
-    <limit effort="${motor_stall_torque}"/>
+    <limit effort="${motor_stall_torque}" velocity="1.0"/>
   </joint>
   <link name="wheel_right_link">
